Commit message: Update "pioneer_arm" stack for ROS electric
git-svn-id: https://gt-ros-pkg.googlecode.com/svn/trunk@2104 5fc10e88-4e10-11de-b850-9977aa68d080

File: humans/pioneer_arm/pioneer_arm_description/urdf/pioneer_arm.controller.xacro (robot description, xacro)
@@ -32,7 +32,6 @@
 				<interface:audio name="actuator_array_iface"/>
 				<alwaysOn>true</alwaysOn>
-				<updateRate>1000.0</updateRate>
+				<updateRate>10.0</updateRate>
 				<robotParam>${robot_description}</robotParam>
-				<actuatorNamespace>arm</actuatorNamespace>
 				<joint>
 					<name>Joint0</name>
@@ -45,5 +44,5 @@
 				<joint>
 					<name>Joint1</name>
-					<home>2.3561944902</home>
+					<home>2.094395102</home>
 					<p>10.0</p>
 					<i>0.0</i>
@@ -53,5 +52,5 @@
 				<joint>
 					<name>Joint2</name>
-					<home>1.570796327</home>
+					<home>1.483529864</home>
 					<p>10.0</p>
 					<i>0.0</i>

File: humans/pioneer_arm/pioneer_arm_description/urdf/pioneer_arm.urdf.xacro (robot description, xacro)
@@ -65,5 +65,5 @@
 			<child link="Link1" />
 			<axis xyz="0 0 -1" />
-			<limit lower="-1.5707963268" upper="1.5707963268" effort="100.0" velocity="0.7853981634" />
+			<limit lower="-1.5707963268" upper="1.5707963268" effort="10.0" velocity="15.71" />
 			<dynamics damping="0.0" friction="0.0" />
 		</joint>
@@ -94,5 +94,5 @@
 			<child link="Link2" />
 			<axis xyz="0 -1 0" />
-			<limit lower="-1.308996939" upper="2.3561944902" effort="100.0" velocity="0.7853981634" />
+			<limit lower="-1.308996939" upper="2.3561944902" effort="10.0" velocity="15.71" />
 			<dynamics damping="0.0" friction="0.0" />
 		</joint>
@@ -123,5 +123,5 @@
 			<child link="Link3" />
 			<axis xyz="0 -1 0" />
-			<limit lower="-2.0943951024" upper="1.5707963268" effort="100.0" velocity="0.7853981634" />
+			<limit lower="-2.0943951024" upper="1.5707963268" effort="10.0" velocity="15.71" />
 			<dynamics damping="0.0" friction="0.0" />
 		</joint>
@@ -152,5 +152,5 @@
 			<child link="Link4" />
 			<axis xyz="1 0 0" />
-			<limit lower="-1.5707963268" upper="1.5707963268" effort="100.0" velocity="0.7853981634" />
+			<limit lower="-1.5707963268" upper="1.5707963268" effort="10.0" velocity="15.71" />
 			<dynamics damping="0.0" friction="0.0" />
 		</joint>
@@ -181,5 +181,5 @@
 			<child link="Link5" />
 			<axis xyz="0 1 0" />
-			<limit lower="-1.5707963268" upper="1.5707963268" effort="100.0" velocity="0.7853981634" />
+			<limit lower="-1.5707963268" upper="1.5707963268" effort="10.0" velocity="15.71" />
 			<dynamics damping="0.0" friction="0.0" />
 		</joint>
@@ -210,5 +210,5 @@
 			<child link="GripperLink" />
 			<axis xyz="0 0 1" />
-			<limit lower="-0.5235987756" upper="1.2217304764" effort="100.0" velocity="0.7853981634" />
+			<limit lower="-0.5235987756" upper="1.2217304764" effort="10.0" velocity="15.71" />
 			<dynamics damping="0.0" friction="0.0" />
 		</joint>
@@ -235,9 +235,9 @@
 		</link>
         <joint name="RightGripperJoint" type="prismatic">
-			<origin xyz=" 0.10000 -0.01060  0.00000" rpy=" 0.00000  0.00000  0.00000" />
+			<origin xyz=" 0.09275 -0.01060  0.00000" rpy=" 0.00000  0.00000  0.00000" />
 			<parent link="Link5" />
 			<child link="RightGripper" />
 			<axis xyz="0 -1 0" />
-			<limit lower="0.0" upper="0.026" effort="100.0" velocity="0.0117" />
+			<limit lower="0.0" upper="0.026" effort="1.0" velocity="0.2340" />
 			<dynamics damping="0" friction="0" />
 			<mimic joint="Joint5" multiplier="0.0148969027" offset="-0.5235987756"/>
@@ -265,9 +265,9 @@
 		</link>
         <joint name="LeftGripperJoint" type="prismatic">
-			<origin xyz=" 0.10000  0.01060  0.00000" rpy=" 0.00000  0.00000  0.00000" />
+			<origin xyz=" 0.09275  0.01060  0.00000" rpy=" 0.00000  0.00000  0.00000" />
 			<parent link="Link5" />
 			<child link="LeftGripper" />
 			<axis xyz="0 1 0" />
-			<limit lower="0.0" upper="0.026" effort="1.0" velocity="0.0117" />
+			<limit lower="0.0" upper="0.026" effort="1.0" velocity="0.2340" />
 			<dynamics damping="0" friction="0" />
 			<mimic joint="Joint5" multiplier="0.0148969027" offset="-0.5235987756"/>
