Commit message: Fixed coordinates on example arm urdf
git-svn-id: https://gt-ros-pkg.googlecode.com/svn/trunk@2745 5fc10e88-4e10-11de-b850-9977aa68d080

File: humans/actuator_array/actuator_array_example/robots/example_arm.urdf (robot description, URDF)
Before this commit: robot example_arm, 5 links, 4 joints
Links:
- link link1: geometry collision cylinder length=0.02000 radius=0.05000; visual cylinder length=0.02000 radius=0.05000
- link link2: mass 0.30 -> 0.10; geometry collision box size=0.20000 0.02000 0.02000; visual box size=0.20000 0.02000 0.02000
- link link3: geometry collision box size=0.20000 0.02000 0.02000; visual box size=0.20000 0.02000 0.02000
- link link4: geometry collision box size=0.20000 0.02000 0.02000; visual box size=0.20000 0.02000 0.02000
Joints:
- joint joint1: limit lower=${-pi/2} upper=${pi/2} effort=10.0 velocity=15.71 -> lower=-1.57 upper=+1.57 effort=10.0 velocity=15.71
- joint joint2: limit lower=${-pi} upper=0.00000 effort=10.0 velocity=15.71 -> lower=-3.14 upper=0.0 effort=10.0 velocity=15.71; origin xyz= 0.00000  0.00000  0.05000 rpy= 0.00000  0.00000  0.00000 -> xyz= 0.00000  0.00000  0.03000 rpy= 0.00000  0.00000  0.00000
- joint joint3: limit lower=0.00000 upper=${pi} effort=10.0 velocity=15.71 -> lower=-1.57 upper=1.57 effort=10.0 velocity=15.71
- joint joint4: limit lower=0.00000 upper=${pi/2} effort=10.0 velocity=15.71 -> lower=-1.57 upper=1.57 effort=10.0 velocity=15.71; origin xyz= 0.10000  0.00000  0.00000 rpy= 0.00000  0.00000  0.00000 -> xyz= 0.20000  0.00000  0.00000 rpy= 0.00000  0.00000  0.00000
